File: development/arena_12-12/teensy4p1/teensy_arena_12-12_v0p1/holes.kicad_sch (KiCad schematic)
At the start: 4 parts

Commit message: bump buffer version to 0.2
Other:
- moved on the sheet: H1, H2, H3, H4
