File: development/arena_12-12/teensy4p1/teensy_arena_12-12_v0p1/level_shifters.kicad_sch (KiCad schematic)
At the start: 166 parts, among them U10 TXB0108PW, U11 TXB0108PW, U12 TXB0108PW, U13 TXB0108PW, U14 TXB0108PW, U15 74LVC1G17, U16 74LVC1G17, U17 74LVC1G17, U18 74LVC1G17, U19 74LVC2G17, U20 74LVC2G17, U21 74LVC2G17, U22 74LVC2G17, U23 74LVC2G17, U24 74LVC2G17, U25 74LVC2G17, U26 74LVC2G17, U27 74LVC2G17, U28 74LVC2G17, U29 74LVC2G17, U3 TXB0108PW, U30 74LVC2G17, U31 74LVC2G17, U32 74LVC2G17, U33 74LVC2G17, U34 74LVC2G17, U35 74LVC2G17, U4 TXB0108PW, U5 TXB0108PW, U6 TXB0108PW, U7 TXB0108PW, U8 TXB0108PW, U9 TXB0108PW

Commit message: bump buffer version to 0.2
Parts:
- removed C12, C13, C14, C15, C16, C17, C18, C19, C20, C21, C22, C23, C24, C25, C26, C27, C28, C29, C30, C31, C32, C33, C34, C35, C36, C37, C38, C39, C40, C41, C42, C43, C44, C45, C46: 0.1uF, Capacitor_SMD:C_0402_1005Metric, symbol Device:C
- removed R100, R101, R102, R103, R104, R105, R106, R107, R108, R109, R110, R111, R112, R113, R114, R115, R116, R117, R118, R119, R120, R121, R122, R123, R124, R125, R126, R39, R40, R41, R42, R43, R44, R45, R46, R47, R48, R49, R50, R51, R52, R53, R54, R55, R56, R57, R58, R59, R60, R61, R62, R63, R64, R65, R66, R67, R68, R69, R70, R71, R72, R73, R74, R75, R76, R77, R78, R79, R80, R81, R82, R83, R84, R85, R86, R87, R88, R89, R90, R91, R92, R93, R94, R95, R96, R97, R98, R99: 33, Resistor_SMD:R_0402_1005Metric, symbol Device:R
- removed U10, U11, U12, U13, U14, U6, U7, U8, U9: TXB0108PW, Package_SO:TSSOP-20_4.4x6.5mm_P0.65mm, symbol TXB0108:TXB0108PW
- removed U15, U16, U17, U18: 74LVC1G17, Package_TO_SOT_SMD:SOT-23-5, symbol 74xGxx:74LVC1G17
- removed U19, U20, U21, U22, U23, U24, U25, U26, U27, U28, U29, U30, U31, U32, U33, U34, U35: 74LVC2G17, Package_TO_SOT_SMD:SOT-23-6, symbol 74xGxx:74LVC2G17
- added U4, U5: TXB0108PW, Package_SO:TSSOP-20_4.4x6.5mm_P0.65mm, symbol TXB0108:TXB0108PW
- C1: renamed from C2; footprint Capacitor_SMD:C_0402_1005Metric -> Capacitor_SMD:C_0603_1608Metric
- C10: renamed from C11; footprint Capacitor_SMD:C_0402_1005Metric -> Capacitor_SMD:C_0603_1608Metric
- C2: renamed from C3; footprint Capacitor_SMD:C_0402_1005Metric -> Capacitor_SMD:C_0603_1608Metric
- C3: renamed from C4; footprint Capacitor_SMD:C_0402_1005Metric -> Capacitor_SMD:C_0603_1608Metric
- C4: renamed from C5; footprint Capacitor_SMD:C_0402_1005Metric -> Capacitor_SMD:C_0603_1608Metric
- C5: renamed from C6; footprint Capacitor_SMD:C_0402_1005Metric -> Capacitor_SMD:C_0603_1608Metric
- C6: renamed from C7; footprint Capacitor_SMD:C_0402_1005Metric -> Capacitor_SMD:C_0603_1608Metric
- C7: renamed from C8; footprint Capacitor_SMD:C_0402_1005Metric -> Capacitor_SMD:C_0603_1608Metric
- C8: renamed from C9; footprint Capacitor_SMD:C_0402_1005Metric -> Capacitor_SMD:C_0603_1608Metric
- C9: renamed from C10; footprint Capacitor_SMD:C_0402_1005Metric -> Capacitor_SMD:C_0603_1608Metric
- renumbered U3 to U1, U4 to U2, U5 to U3
Connections:
- net +3.3V: now also U4.10 (OE), U4.2 (VCCA), U5.10 (OE), U5.2 (VCCA)
- net +5V: now also U4.19 (VCCB), U5.19 (VCCB)
- net GND: now also U4.11 (GND), U5.11 (GND)
- net PAN3V.CS_00: now also U2.1 (A1)
- net PAN3V.CS_01: now also U2.3 (A2)
- net PAN3V.CS_02: now also U2.4 (A3)
- net PAN3V.CS_03: now also U2.5 (A4)
- net PAN3V.CS_04: now also U2.6 (A5)
- net PAN3V.CS_05: now also U2.7 (A6)
- net PAN3V.CS_06: now also U2.8 (A7)
- net PAN3V.CS_07: now also U2.9 (A8)
- net PAN3V.CS_08: now also U3.1 (A1)
- net PAN3V.CS_09: now also U3.3 (A2)
- net PAN3V.CS_10: now also U3.4 (A3)
- net PAN3V.CS_11: now also U3.5 (A4)
- net PAN3V.CS_12: now also U3.6 (A5)
- net PAN3V.CS_13: now also U3.7 (A6)
- net PAN3V.CS_14: now also U3.8 (A7)
- net PAN3V.CS_15: now also U3.9 (A8)
- net PAN3V.CS_16: now also U4.1 (A1)
- net PAN3V.CS_17: now also U4.3 (A2)
- net PAN3V.CS_18: now also U4.4 (A3)
- net PAN3V.CS_19: now also U4.5 (A4)
- net PAN3V.CS_20: now also U4.6 (A5)
- net PAN3V.CS_21: now also U4.7 (A6)
- net PAN3V.CS_22: now also U4.8 (A7)
- net PAN3V.CS_23: now also U4.9 (A8)
- net PAN3V.CS_24: now also U5.1 (A1)
- net PAN3V.CS_25: now also U5.3 (A2)
- net PAN3V.CS_26: now also U5.4 (A3)
- net PAN3V.CS_27: now also U5.5 (A4)
- net PAN3V.CS_28: now also U5.6 (A5)
- net PAN3V.CS_29: now also U5.7 (A6)
- net PAN3V.EXT_INT: now also U5.9 (A8)
- net PAN3V.MISO_0: now also U1.5 (A4)
- net PAN3V.MISO_1: now also U1.9 (A8)
- net PAN3V.MOSI_0: now also U1.4 (A3)
- net PAN3V.MOSI_1: now also U1.8 (A7)
- net PAN3V.RESET: now also U1.1 (A1)
- net PAN3V.SCK_0: now also U1.3 (A2)
- net PAN3V.SCK_1: now also U1.7 (A6)
- net PAN5V.EXT_INT: now also U5.12 (B8)
- net PAN5V.MISO_0: now also U1.16 (B4)
- net PAN5V.MISO_1: now also U1.12 (B8)
- net PAN5V.RESET: now also U1.20 (B1)
- net PAN5V.CS_11: now reaches U3.16 (B4)
- net PAN5V.MOSI_1: now reaches U1.13 (B7)
- net PAN5V.CS_01: now reaches U2.18 (B2)
- net PAN5V.SCK_1: now reaches U1.14 (B6)
- net PAN5V.MOSI_0: now reaches U1.17 (B3)
- net PAN5V.SCK_0: now reaches U1.18 (B2)
- net PAN5V.CS_05: now reaches U2.14 (B6)
- net PAN5V.CS_09: now reaches U3.18 (B2)
- net PAN5V.CS_08: now reaches U3.20 (B1)
- net PAN5V.CS_15: now reaches U3.12 (B8)
- net PAN5V.CS_03: now reaches U2.16 (B4)
- net PAN5V.CS_14: now reaches U3.13 (B7)
- net PAN5V.CS_07: now reaches U2.12 (B8)
- net PAN5V.CS_13: now reaches U3.14 (B6)
- net PAN5V.CS_06: now reaches U2.13 (B7)
- net PAN5V.CS_04: now reaches U2.15 (B5)
- net PAN5V.CS_02: now reaches U2.17 (B3)
- net PAN5V.CS_00: now reaches U2.20 (B1)
- net PAN5V.CS_12: now reaches U3.15 (B5)
- net PAN5V.CS_10: now reaches U3.17 (B3)
- new net PAN5V.CS_16: U4.20 (B1)
- new net PAN5V.CS_17: U4.18 (B2)
- new net PAN5V.CS_18: U4.17 (B3)
- new net PAN5V.CS_19: U4.16 (B4)
- new net PAN5V.CS_20: U4.15 (B5)
- new net PAN5V.CS_21: U4.14 (B6)
- new net PAN5V.CS_22: U4.13 (B7)
- new net PAN5V.CS_23: U4.12 (B8)
- new net PAN5V.CS_24: U5.20 (B1)
- new net PAN5V.CS_25: U5.18 (B2)
- new net PAN5V.CS_26: U5.17 (B3)
- new net PAN5V.CS_27: U5.16 (B4)
- new net PAN5V.CS_28: U5.15 (B5)
- new net PAN5V.CS_29: U5.14 (B6)
- no-connect marks 20 -> 4
Other:
- note removed: "SN74LVC1G17DBVR C7836"
- moved on the sheet: C1, C10, C2, C3, C4, C5, C6, C7, C8, C9, U1, U2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
