File: development/arena_12-12/teensy4p1/teensy_arena_12-12_v0p1/panel_headers.kicad_sch (KiCad schematic)
At the start: 231 parts, among them P1 CONN15, P10 CONN15, P11 CONN15, P12 CONN15, P2 CONN15, P3 CONN15, P4 CONN15, P5 CONN15, P6 CONN15, P7 CONN15, P8 CONN15, P9 CONN15, Q1 MOSFET_NCHAN, U36 74LVC2G17, U37 74LVC2G17, U38 74LVC2G17, U39 74LVC2G17, U40 74LVC2G17, U41 74LVC2G17, U42 74LVC2G17, U43 74LVC2G17, U44 74LVC2G17, U45 74LVC2G17, U46 74LVC2G17, U47 74LVC2G17, U48 74LVC2G17, U49 74LVC2G17, U50 74LVC2G17, U51 74LVC2G17, U52 74LVC2G17, U53 74LVC2G17, U54 74LVC2G17, U55 74LVC2G17, U56 74LVC2G17, U57 74LVC2G17, U58 74LVC2G17, U59 74LVC2G17, U60 74LVC2G17, U61 74LVC2G17, U62 74LVC2G17, U63 74LVC2G17, U64 74LVC2G17, U65 74LVC2G17, U66 74LVC2G17, U67 74LVC2G17, U68 74LVC2G17, U69 74LVC2G17, U70 74LVC2G17, U71 74LVC2G17, U72 74LVC2G17, U73 74LVC2G17, U74 74LVC2G17, U75 74LVC2G17, U76 74LVC2G17, U77 74LVC2G17, U78 74LVC2G17, U79 74LVC2G17, U80 74LVC2G17, U81 74LVC2G17, U82 74LVC2G17, U83 74LVC2G17

Commit message: bump buffer version to 0.2
Parts:
- removed C47, C48, C49, C50, C51, C52, C53, C54, C55, C56, C57, C58, C59, C60, C61, C62, C63, C64, C65, C66, C67, C68, C69, C70, C71, C72, C73, C74, C75, C76, C77, C78, C79, C80, C81, C82, C83, C84, C85, C86, C87, C88, C89, C90, C91, C92, C93, C94: 0.1uF, Capacitor_SMD:C_0402_1005Metric, symbol Device:C
- removed Q1: MOSFET_NCHAN, Package_TO_SOT_SMD:SOT-23-3, symbol arena_custom:MOSFET_NCHAN
- removed R127, R128, R129, R130, R131, R132, R133, R134, R135, R136, R137, R138, R139, R140, R141, R142, R143, R144, R145, R146, R147, R148, R149, R150, R151, R152, R153, R154, R155, R156, R157, R158, R159, R160, R161, R162, R163, R164, R165, R166, R167, R168, R169, R170, R171, R172, R173, R174, R175, R176, R177, R178, R179, R180, R181, R182, R183, R184, R185, R186, R187, R188, R189, R190, R191, R192, R193, R194, R195, R196, R197, R198, R199, R200, R201, R202, R203, R204, R205, R206, R207, R208, R209, R210, R211, R212, R213, R214, R215, R216, R217, R218, R219, R220, R221, R222, R223, R224, R225, R226, R227, R228, R229, R230, R231, R232, R233, R234: 33, Resistor_SMD:R_0402_1005Metric, symbol Device:R
- removed U36, U37, U38, U39, U40, U41, U42, U43, U44, U45, U46, U47, U48, U49, U50, U51, U52, U53, U54, U55, U56, U57, U58, U59, U60, U61, U62, U63, U64, U65, U66, U67, U68, U69, U70, U71, U72, U73, U74, U75, U76, U77, U78, U79, U80, U81, U82, U83: 74LVC2G17, Package_TO_SOT_SMD:SOT-23-6, symbol 74xGxx:74LVC2G17
- added Q2: MOSFET_NCHAN, Package_TO_SOT_SMD:SOT-23-3, symbol arena_custom:MOSFET_NCHAN
- R1, R2: footprint Resistor_SMD:R_0402_1005Metric -> Resistor_SMD:R_0805_2012Metric
- renumbered C95 to C11, C96 to C12, C97 to C13, C98 to C14, C99 to C15, C100 to C16, C101 to C17, C102 to C18, C103 to C19, C104 to C20, C105 to C21, C106 to C22
Connections:
- net HDR_CS_00_P7 is gone; now on net PAN5V.CS_00: P7.7
- net HDR_CS_01_P7 is gone; now on net PAN5V.CS_01: P7.8
- net HDR_CS_02_P7 is gone; now on net PAN5V.CS_02: P7.9
- net HDR_CS_03_P7 is gone; now on net PAN5V.CS_03: P7.10
- net HDR_CS_04_P7 is gone; now on net PAN5V.CS_04: P7.11
- net HDR_CS_05_P8 is gone; now on net PAN5V.CS_05: P8.7
- net HDR_CS_06_P8 is gone; now on net PAN5V.CS_06: P8.8
- net HDR_CS_07_P8 is gone; now on net PAN5V.CS_07: P8.9
- net HDR_CS_08_P8 is gone; now on net PAN5V.CS_08: P8.10
- net HDR_CS_09_P8 is gone; now on net PAN5V.CS_09: P8.11
- net HDR_CS_10_P9 is gone; now on net PAN5V.CS_10: P9.7
- net HDR_CS_11_P9 is gone; now on net PAN5V.CS_11: P9.8
- net HDR_CS_12_P9 is gone; now on net PAN5V.CS_12: P9.9
- net HDR_CS_13_P9 is gone; now on net PAN5V.CS_13: P9.10
- net HDR_CS_14_P9 is gone; now on net PAN5V.CS_14: P9.11
- net HDR_CS_15_P4 is gone; now on net PAN5V.CS_15: P4.7
- net HDR_CS_16_P4 is gone; now on net PAN5V.CS_16: P4.8
- net HDR_CS_17_P4 is gone; now on net PAN5V.CS_17: P4.9
- net HDR_CS_18_P4 is gone; now on net PAN5V.CS_18: P4.10
- net HDR_CS_19_P4 is gone; now on net PAN5V.CS_19: P4.11
- net HDR_CS_20_P5 is gone; now on net PAN5V.CS_20: P5.7
- net HDR_CS_21_P5 is gone; now on net PAN5V.CS_21: P5.8
- net HDR_CS_22_P5 is gone; now on net PAN5V.CS_22: P5.9
- net HDR_CS_23_P5 is gone; now on net PAN5V.CS_23: P5.10
- net HDR_CS_24_P5 is gone; now on net PAN5V.CS_24: P5.11
- net HDR_CS_25_P6 is gone; now on net PAN5V.CS_25: P6.7
- net HDR_CS_26_P6 is gone; now on net PAN5V.CS_26: P6.8
- net HDR_CS_27_P6 is gone; now on net PAN5V.CS_27: P6.9
- net HDR_CS_28_P6 is gone; now on net PAN5V.CS_28: P6.10
- net HDR_CS_29_P6 is gone; now on net PAN5V.CS_29: P6.11
- net HDR_EXT_INT_P1 is gone; now on net PAN5V.EXT_INT: P1.15
- net HDR_EXT_INT_P10 is gone; now on net PAN5V.EXT_INT: P10.15
- net HDR_EXT_INT_P11 is gone; now on net PAN5V.EXT_INT: P11.15
- net HDR_EXT_INT_P12 is gone; now on net PAN5V.EXT_INT: P12.15
- net HDR_EXT_INT_P2 is gone; now on net PAN5V.EXT_INT: P2.15
- net HDR_EXT_INT_P3 is gone; now on net PAN5V.EXT_INT: P3.15
- net HDR_EXT_INT_P4 is gone; now on net PAN5V.EXT_INT: P4.15
- net HDR_EXT_INT_P5 is gone; now on net PAN5V.EXT_INT: P5.15
- net HDR_EXT_INT_P6 is gone; now on net PAN5V.EXT_INT: P6.15
- net HDR_EXT_INT_P7 is gone; now on net PAN5V.EXT_INT: P7.15
- net HDR_EXT_INT_P8 is gone; now on net PAN5V.EXT_INT: P8.15
- net HDR_EXT_INT_P9 is gone; now on net PAN5V.EXT_INT: P9.15
- net HDR_MISO_0_P1 is gone; now on net PAN5V.MISO_0: P1.6
- net HDR_MISO_0_P2 is gone; now on net PAN5V.MISO_0: P2.6
- net HDR_MISO_0_P3 is gone; now on net PAN5V.MISO_0: P3.6
- net HDR_MISO_0_P4 is gone; now on net PAN5V.MISO_0: P4.6
- net HDR_MISO_0_P5 is gone; now on net PAN5V.MISO_0: P5.6
- net HDR_MISO_0_P6 is gone; now on net PAN5V.MISO_0: P6.6
- net HDR_MISO_1_P10 is gone; now on net PAN5V.MISO_1: P10.6
- net HDR_MISO_1_P11 is gone; now on net PAN5V.MISO_1: P11.6
- net HDR_MISO_1_P12 is gone; now on net PAN5V.MISO_1: P12.6
- net HDR_MISO_1_P7 is gone; now on net PAN5V.MISO_1: P7.6
- net HDR_MISO_1_P8 is gone; now on net PAN5V.MISO_1: P8.6
- net HDR_MISO_1_P9 is gone; now on net PAN5V.MISO_1: P9.6
- net HDR_MOSI_0_P2 is gone; now on net PAN5V.MOSI_0: P2.5
- net HDR_MOSI_0_P3 is gone; now on net PAN5V.MOSI_0: P3.5
- net HDR_MOSI_0_P4 is gone; now on net PAN5V.MOSI_0: P4.5
- net HDR_MOSI_0_P5 is gone; now on net PAN5V.MOSI_0: P5.5
- net HDR_MOSI_0_P6 is gone; now on net PAN5V.MOSI_0: P6.5
- net HDR_MOSI_1_P11 is gone; now on net PAN5V.MOSI_1: P11.5
- net HDR_MOSI_1_P12 is gone; now on net PAN5V.MOSI_1: P12.5
- net HDR_MOSI_1_P7 is gone; now on net PAN5V.MOSI_1: P7.5
- net HDR_MOSI_1_P8 is gone; now on net PAN5V.MOSI_1: P8.5
- net HDR_MOSI_1_P9 is gone; now on net PAN5V.MOSI_1: P9.5
- net HDR_SCK_0_P2 is gone; now on net PAN5V.SCK_0: P2.4
- net HDR_SCK_0_P3 is gone; now on net PAN5V.SCK_0: P3.4
- net HDR_SCK_0_P4 is gone; now on net PAN5V.SCK_0: P4.4
- net HDR_SCK_0_P5 is gone; now on net PAN5V.SCK_0: P5.4
- net HDR_SCK_0_P6 is gone; now on net PAN5V.SCK_0: P6.4
- net HDR_SCK_1_P11 is gone; now on net PAN5V.SCK_1: P11.4
- net HDR_SCK_1_P12 is gone; now on net PAN5V.SCK_1: P12.4
- net HDR_SCK_1_P7 is gone; now on net PAN5V.SCK_1: P7.4
- net HDR_SCK_1_P8 is gone; now on net PAN5V.SCK_1: P8.4
- net HDR_SCK_1_P9 is gone; now on net PAN5V.SCK_1: P9.4
- net GND: now also Q2.2 (S)
- net at R1.1, R2.2: now also Q2.1 (G)
- net HDR_CS_00_P1 renamed PAN5V.CS_00
- net HDR_CS_01_P1 renamed PAN5V.CS_01
- net HDR_CS_02_P1 renamed PAN5V.CS_02
- net HDR_CS_03_P1 renamed PAN5V.CS_03
- net HDR_CS_04_P1 renamed PAN5V.CS_04
- net HDR_CS_05_P2 renamed PAN5V.CS_05
- net HDR_CS_06_P2 renamed PAN5V.CS_06
- net HDR_CS_07_P2 renamed PAN5V.CS_07
- net HDR_CS_08_P2 renamed PAN5V.CS_08
- net HDR_CS_09_P2 renamed PAN5V.CS_09
- net HDR_CS_10_P3 renamed PAN5V.CS_10
- net HDR_CS_11_P3 renamed PAN5V.CS_11
- net HDR_CS_12_P3 renamed PAN5V.CS_12
- net HDR_CS_13_P3 renamed PAN5V.CS_13
- net HDR_CS_14_P3 renamed PAN5V.CS_14
- net HDR_CS_15_P10 renamed PAN5V.CS_15
- net HDR_CS_16_P10 renamed PAN5V.CS_16
- net HDR_CS_17_P10 renamed PAN5V.CS_17
- net HDR_CS_18_P10 renamed PAN5V.CS_18
- net HDR_CS_19_P10 renamed PAN5V.CS_19
- net HDR_CS_20_P11 renamed PAN5V.CS_20
- net HDR_CS_21_P11 renamed PAN5V.CS_21
- net HDR_CS_22_P11 renamed PAN5V.CS_22
- net HDR_CS_23_P11 renamed PAN5V.CS_23
- net HDR_CS_24_P11 renamed PAN5V.CS_24
- net HDR_CS_25_P12 renamed PAN5V.CS_25
- net HDR_CS_26_P12 renamed PAN5V.CS_26
- net HDR_CS_27_P12 renamed PAN5V.CS_27
- net HDR_CS_28_P12 renamed PAN5V.CS_28
- net HDR_CS_29_P12 renamed PAN5V.CS_29
- net HDR_MOSI_0_P1 renamed PAN5V.MOSI_0
- net HDR_MOSI_1_P10 renamed PAN5V.MOSI_1
- net HDR_RESET renamed RESET
- net RESET: now also Q2.3 (D)
- net HDR_SCK_0_P1 renamed PAN5V.SCK_0
- net HDR_SCK_1_P10 renamed PAN5V.SCK_1
Other:
- note added: "SI2302-TP Digikey SI2302-TPMSCT-ND LCSC C4748714"
- note removed: "SI2302-TP Digikey SI2302-TPMSCT-ND LCSC C4748714 or ME2306D LCSC C165220"
- note removed: "Swap A and B units for better routing?"
- moved on the sheet: C11, C12, C13, C14, C15, C16, C17, C18, C19, C20, C21, C22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
