File: development/arena_12-12/teensy4p1/teensy_arena_12-12_v0p1/power.kicad_sch (KiCad schematic)
At the start: 3 parts, among them J1 Barrel_Jack, J4 Barrel_Jack, SW1 SW_SPDT

Commit message: bump buffer version to 0.2
Parts:
- removed J4: Barrel_Jack, arena_custom:DCJACK_2PIN_HIGHCURRENT, symbol Connector:Barrel_Jack
Other:
- note removed: "Connection PCB top"
- note removed: "External power supply"
- moved on the sheet: J1, SW1
