File: development/arena_12-12/teensy4p1/teensy_arena_12-12_v0p1/teensy.kicad_sch (KiCad schematic)
At the start: 41 parts, among them J2 Conn_01x04, J3 Conn_01x04, U1 Teensy4.1, U2 74LVC2G17

Commit message: bump buffer version to 0.2
Parts:
- removed C1: 0.1uF, Capacitor_SMD:C_0402_1005Metric, symbol Device:C
- removed R10, R11, R12, R13, R14, R15, R16, R17, R18, R19, R20, R21, R22, R23, R24, R25, R26, R27, R28, R29, R3, R30, R31, R32, R33, R34, R35, R36, R37, R38, R4, R5, R6, R7, R8, R9: 33, Resistor_SMD:R_0402_1005Metric, symbol Device:R
- removed U2: 74LVC2G17, Package_TO_SOT_SMD:SOT-23-6, symbol 74xGxx:74LVC2G17
- U18: renamed from U1; footprint teensy:Teensy41_outer_only -> teensy:Teensy41
Connections:
- net TNY_CS_00 is gone; now on net PAN3V.CS_00: U18.2 (0_RX1_CRX2_CS1)
- net TNY_CS_01 is gone; now on net PAN3V.CS_01: U18.4 (2_OUT2)
- net TNY_CS_02 is gone; now on net PAN3V.CS_02: U18.5 (3_LRCLK2)
- net TNY_CS_03 is gone; now on net PAN3V.CS_03: U18.6 (4_BCLK2)
- net TNY_CS_04 is gone; now on net PAN3V.CS_04: U18.7 (5_IN2)
- net TNY_CS_05 is gone; now on net PAN3V.CS_05: U18.8 (6_OUT1D)
- net TNY_CS_06 is gone; now on net PAN3V.CS_06: U18.9 (7_RX2_OUT1A)
- net TNY_CS_07 is gone; now on net PAN3V.CS_07: U18.10 (8_TX2_IN1)
- net TNY_CS_08 is gone; now on net PAN3V.CS_08: U18.11 (9_OUT1C)
- net TNY_CS_09 is gone; now on net PAN3V.CS_09: U18.12 (10_CS_MQSR)
- net TNY_CS_10 is gone; now on net PAN3V.CS_10: U18.16 (24_A10_TX6_SCL2)
- net TNY_CS_11 is gone; now on net PAN3V.CS_11: U18.17 (25_A11_RX6_SDA2)
- net TNY_CS_12 is gone; now on net PAN3V.CS_12: U18.20 (28_RX7)
- net TNY_CS_13 is gone; now on net PAN3V.CS_13: U18.21 (29_TX7)
- net TNY_CS_14 is gone; now on net PAN3V.CS_14: U18.22 (30_CRX3)
- net TNY_CS_15 is gone; now on net PAN3V.CS_15: U18.23 (31_CTX3)
- net TNY_CS_16 is gone; now on net PAN3V.CS_16: U18.24 (32_OUT1B)
- net TNY_CS_17 is gone; now on net PAN3V.CS_17: U18.45 (23_A9_CRX1_MCLK1)
- net TNY_CS_18 is gone; now on net PAN3V.CS_18: U18.44 (22_A8_CTX1)
- net TNY_CS_19 is gone; now on net PAN3V.CS_19: U18.43 (21_A7_RX5_BCLK1)
- net TNY_CS_20 is gone; now on net PAN3V.CS_20: U18.42 (20_A6_TX5_LRCLK1)
- net TNY_CS_21 is gone; now on net PAN3V.CS_21: U18.39 (17_A3_TX4_SDA1)
- net TNY_CS_22 is gone; now on net PAN3V.CS_22: U18.38 (16_A2_RX4_SCL1)
- net TNY_CS_23 is gone; now on net PAN3V.CS_23: U18.33 (41_A17)
- net TNY_CS_24 is gone; now on net PAN3V.CS_24: U18.32 (40_A16)
- net TNY_CS_25 is gone; now on net PAN3V.CS_25: U18.31 (39_MISO1_OUT1A)
- net TNY_CS_26 is gone; now on net PAN3V.CS_26: U18.30 (38_CS1_IN1)
- net TNY_CS_27 is gone; now on net PAN3V.CS_27: U18.29 (37_CS)
- net TNY_CS_28 is gone; now on net PAN3V.CS_28: U18.28 (36_CS)
- net TNY_CS_29 is gone; now on net PAN3V.CS_29: U18.27 (35_TX8)
- net TNY_EXT_INT is gone; now on net PAN3V.EXT_INT: U18.25 (33_MCLK2)
- net TNY_MISO_0 is gone; now on net PAN3V.MISO_0: U18.14 (12_MISO_MQSL)
- net TNY_MISO_1 is gone; now on net PAN3V.MISO_1: U18.3 (1_TX1_CTX2_MISO1)
- net TNY_MOSI_0 is gone; now on net PAN3V.MOSI_0: U18.13 (11_MOSI_CTX1)
- net TNY_MOSI_1 is gone; now on net PAN3V.MOSI_1: U18.18 (26_A12_MOSI1)
- net TNY_RESET is gone; now on net PAN3V.RESET: U18.26 (34_RX8)
- net TNY_SCK_0 is gone; now on net PAN3V.SCK_0: U18.35 (13_SCK_LED)
- net TNY_SCK_1 is gone; now on net PAN3V.SCK_1: U18.19 (27_A13_SCK1)
- no-connect marks 1 -> 20
Other:
- note removed: "SN74LVC2G17DBVR C10429"
- moved on the sheet: J2, J3
