File: development/arena_12-12/teensy4p1/teensy_arena_12-12_v0p1/teensy_arena_12-12.kicad_sch (KiCad schematic)
At the start: 0 parts

Commit message: bump buffer version to 0.2
Other:
- sheet Level Shifters ports: added PAN3V{PAN}, PAN5V{PAN}; removed PAN3V{PAN3V}, PAN5V{PAN5V}
- sheet Panel Headers ports: added PAN5V{PAN}; removed PAN5V{PAN5V}
- sheet Teensy ports: added PAN3V{PAN}; removed PAN3V{PAN3V}
