File: development/arena_12-12/teensy4p1/teensy_arena_12-12_v0p1/layout_tool/modified_teensy_arena_12-12.kicad_pcb (KiCad board)
At the start: 6 copper layers, 228.6 x 228.6 mm, 445 parts, among them J1 Barrel_Jack, J2 Conn_01x04, J3 Conn_01x04, J4 Barrel_Jack, P1 CONN15, P10 CONN15, P11 CONN15, P12 CONN15, P2 CONN15, P3 CONN15, P4 CONN15, P5 CONN15, P6 CONN15, P7 CONN15, P8 CONN15, P9 CONN15, Q1 MOSFET_NCHAN, SW1 SW_SPDT, U1 Teensy4.1, U10 TXB0108PW, U11 TXB0108PW, U12 TXB0108PW, U13 TXB0108PW, U14 TXB0108PW, U15 74LVC1G17, U16 74LVC1G17, U17 74LVC1G17, U18 74LVC1G17, U19 74LVC2G17, U2 74LVC2G17, U20 74LVC2G17, U21 74LVC2G17, U22 74LVC2G17, U23 74LVC2G17, U24 74LVC2G17, U25 74LVC2G17, U26 74LVC2G17, U27 74LVC2G17, U28 74LVC2G17, U29 74LVC2G17, U3 TXB0108PW, U30 74LVC2G17, U31 74LVC2G17, U32 74LVC2G17, U33 74LVC2G17, U34 74LVC2G17, U35 74LVC2G17, U36 74LVC2G17, U37 74LVC2G17, U38 74LVC2G17, U39 74LVC2G17, U4 TXB0108PW, U40 74LVC2G17, U41 74LVC2G17, U42 74LVC2G17, U43 74LVC2G17, U44 74LVC2G17, U45 74LVC2G17, U46 74LVC2G17, U47 74LVC2G17, U48 74LVC2G17, U49 74LVC2G17, U5 TXB0108PW, U50 74LVC2G17, U51 74LVC2G17, U52 74LVC2G17, U53 74LVC2G17, U54 74LVC2G17, U55 74LVC2G17, U56 74LVC2G17, U57 74LVC2G17, U58 74LVC2G17, U59 74LVC2G17, U6 TXB0108PW, U60 74LVC2G17, U61 74LVC2G17, U62 74LVC2G17, U63 74LVC2G17, U64 74LVC2G17, U65 74LVC2G17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

Commit message: bump buffer version to 0.2
Parts:
- removed the C11 at (-71.9, 138.1)
- removed the C12 at (-71.9, 140.6)
- removed the C13 at (-71.9, 143.1)
- removed the C14 at (-71.9, 145.6)
- removed the C15 at (-71.9, 148.1)
- removed the C16 at (-71.9, 150.6)
- removed the C17 at (-67.9, 115.5)
- removed the C18 at (-67.9, 118.0)
- removed the C19 at (-67.9, 120.5)
- removed the C20 at (-67.9, 123.0)
- removed the C21 at (-67.9, 125.5)
- removed the C22 at (-67.9, 128.0)
- removed C23, C24, C25, C26, C27, C28, C29, C30, C31, C32, C33, C34, C35, C36, C37, C38, C39, C40, C41, C42, C43, C44, C45, C46, C47, C48, C49, C50, C51, C52, C53, C54, C55, C56, C57, C58, C59, C60, C61, C62, C63, C64, C65, C66, C67, C68, C69, C70, C71, C72, C73, C74, C75, C76, C77, C78, C79, C80, C81, C82, C83, C84, C85, C86, C87, C88, C89, C90, C91, C92, C93, C94: 0.1uF, Capacitor_SMD:C_0402_1005Metric
- removed J4: Barrel_Jack, arena_custom:DCJACK_2PIN_HIGHCURRENT
- removed Q1: MOSFET_NCHAN, Package_TO_SOT_SMD:SOT-23-3
- removed R10, R100, R101, R102, R103, R104, R105, R106, R107, R108, R109, R11, R110, R111, R112, R113, R114, R115, R116, R117, R118, R119, R12, R120, R121, R122, R123, R124, R125, R126, R127, R128, R129, R13, R130, R131, R132, R133, R134, R135, R136, R137, R138, R139, R14, R140, R141, R142, R143, R144, R145, R146, R147, R148, R149, R15, R150, R151, R152, R153, R154, R155, R156, R157, R158, R159, R16, R160, R161, R162, R163, R164, R165, R166, R167, R168, R169, R17, R170, R171, R172, R173, R174, R175, R176, R177, R178, R179, R18, R180, R181, R182, R183, R184, R185, R186, R187, R188, R189, R19, R190, R191, R192, R193, R194, R195, R196, R197, R198, R199, R20, R200, R201, R202, R203, R204, R205, R206, R207, R208, R209, R21, R210, R211, R212, R213, R214, R215, R216, R217, R218, R219, R22, R220, R221, R222, R223, R224, R225, R226, R227, R228, R229, R23, R230, R231, R232, R233, R234, R24, R25, R26, R27, R28, R29, R3, R30, R31, R32, R33, R34, R35, R36, R37, R38, R39, R4, R40, R41, R42, R43, R44, R45, R46, R47, R48, R49, R5, R50, R51, R52, R53, R54, R55, R56, R57, R58, R59, R6, R60, R61, R62, R63, R64, R65, R66, R67, R68, R69, R7, R70, R71, R72, R73, R74, R75, R76, R77, R78, R79, R8, R80, R81, R82, R83, R84, R85, R86, R87, R88, R89, R9, R90, R91, R92, R93, R94, R95, R96, R97, R98, R99: 68, Resistor_SMD:R_0402_1005Metric
- removed U10, U11, U12, U13, U14, U6, U7, U8, U9: TXB0108PW, Package_SO:TSSOP-20_4.4x6.5mm_P0.65mm
- removed U15, U16, U17: 74LVC1G17, Package_TO_SOT_SMD:SOT-23-5
- removed the U18 at (-35.2, 129.8)
- removed U19, U20, U21, U22, U23, U24, U25, U26, U27, U28, U29, U30, U31, U32, U33, U34, U35, U36, U37, U38, U39, U40, U41, U42, U43, U44, U45, U46, U47, U48, U49, U50, U51, U52, U53, U54, U55, U56, U57, U58, U59, U60, U61, U62, U63, U64, U65, U66, U67, U68, U69, U70, U71, U72, U73, U74, U75, U76, U77, U78, U79, U80, U81, U82, U83: 74LVC2G17, Package_TO_SOT_SMD:SOT-23-6
- added Q2: MOSFET_NCHAN, Package_TO_SOT_SMD:SOT-23-3, F.Cu at (291.5, 164.3)
- added U1: TXB0108PW, Package_SO:TSSOP-20_4.4x6.5mm_P0.65mm, F.Cu at (280.9, 222.8)
- C1, C10, C2, C3, C4, C5, C6, C7, C8, C9: footprint Capacitor_SMD:C_0402_1005Metric -> Capacitor_SMD:C_0603_1608Metric
- U2: value 74LVC2G17 -> TXB0108PW; footprint Package_TO_SOT_SMD:SOT-23-6 -> Package_SO:TSSOP-20_4.4x6.5mm_P0.65mm
- moved C7 383.7 mm to (274.3, 293.6)
- moved C8 371.5 mm to (261.9, 293.7), turned to 180 degrees
- moved C6 340.6 mm to (224.4, 293.7), turned to 180 degrees
- moved C9 309.3 mm to (192.5, 293.6)
- moved C10 297.6 mm to (180.4, 293.6), turned to 180 degrees
- moved U5 282.4 mm to (186.5, 291.3), turned to 180 degrees
- moved C2 261.7 mm to (287.3, 220.5), turned to 0 degrees
- moved C3 233.0 mm to (274.5, 239.1), turned to 180 degrees
- moved C4 218.8 mm to (286.9, 239.1), turned to 0 degrees
- moved U3 184.6 mm to (230.5, 291.4), turned to 180 degrees
- moved U4 183.6 mm to (268.0, 291.4), turned to 180 degrees
- moved C5 146.4 mm to (236.7, 293.7)
- moved J2 78.2 mm to (301.5, 239.5)
- moved J3 78.2 mm to (301.5, 230.5)
- moved C1 46.6 mm to (273.9, 220.5), turned to 180 degrees
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- renumbered C95 to C11, C96 to C12, C97 to C13, C98 to C14, C99 to C15, C100 to C16, C101 to C17, C102 to C18, C103 to C19, C104 to C20, C105 to C21, C106 to C22, U1 to U18
Connections:
- net /Panel Headers/HDR_RESET renamed /Panel Headers/RESET
- net /Power/SW_5V renamed Net-(SW1-A)
- C10 pad 1: +3.3V -> +5V
- C2 pad 1: +3.3V -> +5V
- C3 pad 1: +5V -> +3.3V
- C4 pad 1: +3.3V -> +5V
- C5 pad 1: +5V -> +3.3V
- C6 pad 1: +3.3V -> +5V
- C7 pad 1: +5V -> +3.3V
- C8 pad 1: +3.3V -> +5V
- C9 pad 1: +5V -> +3.3V
- P1 pad 10: /Panel Headers/HDR_CS_03_P1 -> /Level Shifters/PAN5V.CS_03
- P1 pad 11: /Panel Headers/HDR_CS_04_P1 -> /Level Shifters/PAN5V.CS_04
- P1 pad 15: /Panel Headers/HDR_EXT_INT_P1 -> /Level Shifters/PAN5V.EXT_INT
- P1 pad 4: /Panel Headers/HDR_SCK_0_P1 -> /Level Shifters/PAN5V.SCK_0
- P1 pad 5: /Panel Headers/HDR_MOSI_0_P1 -> /Level Shifters/PAN5V.MOSI_0
- P1 pad 6: /Panel Headers/HDR_MISO_0_P1 -> /Level Shifters/PAN5V.MISO_0
- P1 pad 7: /Panel Headers/HDR_CS_00_P1 -> /Level Shifters/PAN5V.CS_00
- P1 pad 8: /Panel Headers/HDR_CS_01_P1 -> /Level Shifters/PAN5V.CS_01
- P1 pad 9: /Panel Headers/HDR_CS_02_P1 -> /Level Shifters/PAN5V.CS_02
- P10 pad 10: /Panel Headers/HDR_CS_18_P10 -> /Level Shifters/PAN5V.CS_18
- P10 pad 11: /Panel Headers/HDR_CS_19_P10 -> /Level Shifters/PAN5V.CS_19
- P10 pad 15: /Panel Headers/HDR_EXT_INT_P10 -> /Level Shifters/PAN5V.EXT_INT
- P10 pad 4: /Panel Headers/HDR_SCK_1_P10 -> /Level Shifters/PAN5V.SCK_1
- P10 pad 5: /Panel Headers/HDR_MOSI_1_P10 -> /Level Shifters/PAN5V.MOSI_1
- P10 pad 6: /Panel Headers/HDR_MISO_1_P10 -> /Level Shifters/PAN5V.MISO_1
- P10 pad 7: /Panel Headers/HDR_CS_15_P10 -> /Level Shifters/PAN5V.CS_15
- P10 pad 8: /Panel Headers/HDR_CS_16_P10 -> /Level Shifters/PAN5V.CS_16
- P10 pad 9: /Panel Headers/HDR_CS_17_P10 -> /Level Shifters/PAN5V.CS_17
- P11 pad 10: /Panel Headers/HDR_CS_23_P11 -> /Level Shifters/PAN5V.CS_23
- P11 pad 11: /Panel Headers/HDR_CS_24_P11 -> /Level Shifters/PAN5V.CS_24
- P11 pad 15: /Panel Headers/HDR_EXT_INT_P11 -> /Level Shifters/PAN5V.EXT_INT
- P11 pad 4: /Panel Headers/HDR_SCK_1_P11 -> /Level Shifters/PAN5V.SCK_1
- P11 pad 5: /Panel Headers/HDR_MOSI_1_P11 -> /Level Shifters/PAN5V.MOSI_1
- P11 pad 6: /Panel Headers/HDR_MISO_1_P11 -> /Level Shifters/PAN5V.MISO_1
- P11 pad 7: /Panel Headers/HDR_CS_20_P11 -> /Level Shifters/PAN5V.CS_20
- P11 pad 8: /Panel Headers/HDR_CS_21_P11 -> /Level Shifters/PAN5V.CS_21
- P11 pad 9: /Panel Headers/HDR_CS_22_P11 -> /Level Shifters/PAN5V.CS_22
- P12 pad 10: /Panel Headers/HDR_CS_28_P12 -> /Level Shifters/PAN5V.CS_28
- P12 pad 11: /Panel Headers/HDR_CS_29_P12 -> /Level Shifters/PAN5V.CS_29
- P12 pad 15: /Panel Headers/HDR_EXT_INT_P12 -> /Level Shifters/PAN5V.EXT_INT
- P12 pad 4: /Panel Headers/HDR_SCK_1_P12 -> /Level Shifters/PAN5V.SCK_1
- P12 pad 5: /Panel Headers/HDR_MOSI_1_P12 -> /Level Shifters/PAN5V.MOSI_1
- P12 pad 6: /Panel Headers/HDR_MISO_1_P12 -> /Level Shifters/PAN5V.MISO_1
- P12 pad 7: /Panel Headers/HDR_CS_25_P12 -> /Level Shifters/PAN5V.CS_25
- P12 pad 8: /Panel Headers/HDR_CS_26_P12 -> /Level Shifters/PAN5V.CS_26
- P12 pad 9: /Panel Headers/HDR_CS_27_P12 -> /Level Shifters/PAN5V.CS_27
- P2 pad 10: /Panel Headers/HDR_CS_08_P2 -> /Level Shifters/PAN5V.CS_08
- P2 pad 11: /Panel Headers/HDR_CS_09_P2 -> /Level Shifters/PAN5V.CS_09
- P2 pad 15: /Panel Headers/HDR_EXT_INT_P2 -> /Level Shifters/PAN5V.EXT_INT
- P2 pad 4: /Panel Headers/HDR_SCK_0_P2 -> /Level Shifters/PAN5V.SCK_0
- P2 pad 5: /Panel Headers/HDR_MOSI_0_P2 -> /Level Shifters/PAN5V.MOSI_0
- P2 pad 6: /Panel Headers/HDR_MISO_0_P2 -> /Level Shifters/PAN5V.MISO_0
- P2 pad 7: /Panel Headers/HDR_CS_05_P2 -> /Level Shifters/PAN5V.CS_05
- P2 pad 8: /Panel Headers/HDR_CS_06_P2 -> /Level Shifters/PAN5V.CS_06
- P2 pad 9: /Panel Headers/HDR_CS_07_P2 -> /Level Shifters/PAN5V.CS_07
- P3 pad 10: /Panel Headers/HDR_CS_13_P3 -> /Level Shifters/PAN5V.CS_13
- P3 pad 11: /Panel Headers/HDR_CS_14_P3 -> /Level Shifters/PAN5V.CS_14
- P3 pad 15: /Panel Headers/HDR_EXT_INT_P3 -> /Level Shifters/PAN5V.EXT_INT
- P3 pad 4: /Panel Headers/HDR_SCK_0_P3 -> /Level Shifters/PAN5V.SCK_0
- P3 pad 5: /Panel Headers/HDR_MOSI_0_P3 -> /Level Shifters/PAN5V.MOSI_0
- P3 pad 6: /Panel Headers/HDR_MISO_0_P3 -> /Level Shifters/PAN5V.MISO_0
- P3 pad 7: /Panel Headers/HDR_CS_10_P3 -> /Level Shifters/PAN5V.CS_10
- P3 pad 8: /Panel Headers/HDR_CS_11_P3 -> /Level Shifters/PAN5V.CS_11
- P3 pad 9: /Panel Headers/HDR_CS_12_P3 -> /Level Shifters/PAN5V.CS_12
- P4 pad 10: /Panel Headers/HDR_CS_18_P4 -> /Level Shifters/PAN5V.CS_18
- P4 pad 11: /Panel Headers/HDR_CS_19_P4 -> /Level Shifters/PAN5V.CS_19
- P4 pad 15: /Panel Headers/HDR_EXT_INT_P4 -> /Level Shifters/PAN5V.EXT_INT
- P4 pad 4: /Panel Headers/HDR_SCK_0_P4 -> /Level Shifters/PAN5V.SCK_0
- P4 pad 5: /Panel Headers/HDR_MOSI_0_P4 -> /Level Shifters/PAN5V.MOSI_0
- P4 pad 6: /Panel Headers/HDR_MISO_0_P4 -> /Level Shifters/PAN5V.MISO_0
- P4 pad 7: /Panel Headers/HDR_CS_15_P4 -> /Level Shifters/PAN5V.CS_15
- P4 pad 8: /Panel Headers/HDR_CS_16_P4 -> /Level Shifters/PAN5V.CS_16
- P4 pad 9: /Panel Headers/HDR_CS_17_P4 -> /Level Shifters/PAN5V.CS_17
- P5 pad 10: /Panel Headers/HDR_CS_23_P5 -> /Level Shifters/PAN5V.CS_23
- P5 pad 11: /Panel Headers/HDR_CS_24_P5 -> /Level Shifters/PAN5V.CS_24
- P5 pad 15: /Panel Headers/HDR_EXT_INT_P5 -> /Level Shifters/PAN5V.EXT_INT
- P5 pad 4: /Panel Headers/HDR_SCK_0_P5 -> /Level Shifters/PAN5V.SCK_0
- P5 pad 5: /Panel Headers/HDR_MOSI_0_P5 -> /Level Shifters/PAN5V.MOSI_0
- P5 pad 6: /Panel Headers/HDR_MISO_0_P5 -> /Level Shifters/PAN5V.MISO_0
- P5 pad 7: /Panel Headers/HDR_CS_20_P5 -> /Level Shifters/PAN5V.CS_20
- P5 pad 8: /Panel Headers/HDR_CS_21_P5 -> /Level Shifters/PAN5V.CS_21
- P5 pad 9: /Panel Headers/HDR_CS_22_P5 -> /Level Shifters/PAN5V.CS_22
- P6 pad 10: /Panel Headers/HDR_CS_28_P6 -> /Level Shifters/PAN5V.CS_28
- P6 pad 11: /Panel Headers/HDR_CS_29_P6 -> /Level Shifters/PAN5V.CS_29
- P6 pad 15: /Panel Headers/HDR_EXT_INT_P6 -> /Level Shifters/PAN5V.EXT_INT
- P6 pad 4: /Panel Headers/HDR_SCK_0_P6 -> /Level Shifters/PAN5V.SCK_0
- P6 pad 5: /Panel Headers/HDR_MOSI_0_P6 -> /Level Shifters/PAN5V.MOSI_0
- P6 pad 6: /Panel Headers/HDR_MISO_0_P6 -> /Level Shifters/PAN5V.MISO_0
- P6 pad 7: /Panel Headers/HDR_CS_25_P6 -> /Level Shifters/PAN5V.CS_25
- P6 pad 8: /Panel Headers/HDR_CS_26_P6 -> /Level Shifters/PAN5V.CS_26
- P6 pad 9: /Panel Headers/HDR_CS_27_P6 -> /Level Shifters/PAN5V.CS_27
- P7 pad 10: /Panel Headers/HDR_CS_03_P7 -> /Level Shifters/PAN5V.CS_03
- P7 pad 11: /Panel Headers/HDR_CS_04_P7 -> /Level Shifters/PAN5V.CS_04
- P7 pad 15: /Panel Headers/HDR_EXT_INT_P7 -> /Level Shifters/PAN5V.EXT_INT
- P7 pad 4: /Panel Headers/HDR_SCK_1_P7 -> /Level Shifters/PAN5V.SCK_1
- P7 pad 5: /Panel Headers/HDR_MOSI_1_P7 -> /Level Shifters/PAN5V.MOSI_1
- P7 pad 6: /Panel Headers/HDR_MISO_1_P7 -> /Level Shifters/PAN5V.MISO_1
- P7 pad 7: /Panel Headers/HDR_CS_00_P7 -> /Level Shifters/PAN5V.CS_00
- P7 pad 8: /Panel Headers/HDR_CS_01_P7 -> /Level Shifters/PAN5V.CS_01
- P7 pad 9: /Panel Headers/HDR_CS_02_P7 -> /Level Shifters/PAN5V.CS_02
- P8 pad 10: /Panel Headers/HDR_CS_08_P8 -> /Level Shifters/PAN5V.CS_08
- P8 pad 11: /Panel Headers/HDR_CS_09_P8 -> /Level Shifters/PAN5V.CS_09
- P8 pad 15: /Panel Headers/HDR_EXT_INT_P8 -> /Level Shifters/PAN5V.EXT_INT
- P8 pad 4: /Panel Headers/HDR_SCK_1_P8 -> /Level Shifters/PAN5V.SCK_1
- P8 pad 5: /Panel Headers/HDR_MOSI_1_P8 -> /Level Shifters/PAN5V.MOSI_1
- P8 pad 6: /Panel Headers/HDR_MISO_1_P8 -> /Level Shifters/PAN5V.MISO_1
- P8 pad 7: /Panel Headers/HDR_CS_05_P8 -> /Level Shifters/PAN5V.CS_05
- P8 pad 8: /Panel Headers/HDR_CS_06_P8 -> /Level Shifters/PAN5V.CS_06
- P8 pad 9: /Panel Headers/HDR_CS_07_P8 -> /Level Shifters/PAN5V.CS_07
- P9 pad 10: /Panel Headers/HDR_CS_13_P9 -> /Level Shifters/PAN5V.CS_13
- P9 pad 11: /Panel Headers/HDR_CS_14_P9 -> /Level Shifters/PAN5V.CS_14
- P9 pad 15: /Panel Headers/HDR_EXT_INT_P9 -> /Level Shifters/PAN5V.EXT_INT
- P9 pad 4: /Panel Headers/HDR_SCK_1_P9 -> /Level Shifters/PAN5V.SCK_1
- P9 pad 5: /Panel Headers/HDR_MOSI_1_P9 -> /Level Shifters/PAN5V.MOSI_1
- P9 pad 6: /Panel Headers/HDR_MISO_1_P9 -> /Level Shifters/PAN5V.MISO_1
- P9 pad 7: /Panel Headers/HDR_CS_10_P9 -> /Level Shifters/PAN5V.CS_10
- P9 pad 8: /Panel Headers/HDR_CS_11_P9 -> /Level Shifters/PAN5V.CS_11
- P9 pad 9: /Panel Headers/HDR_CS_12_P9 -> /Level Shifters/PAN5V.CS_12
- U18 pad 10: /Teensy/TNY_CS_07 -> /Level Shifters/PAN3V.CS_07
- U18 pad 11: /Teensy/TNY_CS_08 -> /Level Shifters/PAN3V.CS_08
- U18 pad 12: /Teensy/TNY_CS_09 -> /Level Shifters/PAN3V.CS_09
- U18 pad 13: /Teensy/TNY_MOSI_0 -> /Level Shifters/PAN3V.MOSI_0
- U18 pad 14: /Teensy/TNY_MISO_0 -> /Level Shifters/PAN3V.MISO_0
- U18 pad 16: /Teensy/TNY_CS_10 -> /Level Shifters/PAN3V.CS_10
- U18 pad 17: /Teensy/TNY_CS_11 -> /Level Shifters/PAN3V.CS_11
- U18 pad 18: /Teensy/TNY_MOSI_1 -> /Level Shifters/PAN3V.MOSI_1
- U18 pad 19: /Teensy/TNY_SCK_1 -> /Level Shifters/PAN3V.SCK_1
- U18 pad 2: /Teensy/TNY_CS_00 -> /Level Shifters/PAN3V.CS_00
- U18 pad 20: /Teensy/TNY_CS_12 -> /Level Shifters/PAN3V.CS_12
- U18 pad 21: /Teensy/TNY_CS_13 -> /Level Shifters/PAN3V.CS_13
- U18 pad 22: /Teensy/TNY_CS_14 -> /Level Shifters/PAN3V.CS_14
- U18 pad 23: /Teensy/TNY_CS_15 -> /Level Shifters/PAN3V.CS_15
- U18 pad 24: /Teensy/TNY_CS_16 -> /Level Shifters/PAN3V.CS_16
- U18 pad 25: /Teensy/TNY_EXT_INT -> /Level Shifters/PAN3V.EXT_INT
- U18 pad 26: /Teensy/TNY_RESET -> /Level Shifters/PAN3V.RESET
- U18 pad 27: /Teensy/TNY_CS_29 -> /Level Shifters/PAN3V.CS_29
- U18 pad 28: /Teensy/TNY_CS_28 -> /Level Shifters/PAN3V.CS_28
- U18 pad 29: /Teensy/TNY_CS_27 -> /Level Shifters/PAN3V.CS_27
- U18 pad 3: /Teensy/TNY_MISO_1 -> /Level Shifters/PAN3V.MISO_1
- U18 pad 30: /Teensy/TNY_CS_26 -> /Level Shifters/PAN3V.CS_26
- U18 pad 31: /Teensy/TNY_CS_25 -> /Level Shifters/PAN3V.CS_25
- U18 pad 32: /Teensy/TNY_CS_24 -> /Level Shifters/PAN3V.CS_24
- U18 pad 33: /Teensy/TNY_CS_23 -> /Level Shifters/PAN3V.CS_23
- U18 pad 35: /Teensy/TNY_SCK_0 -> /Level Shifters/PAN3V.SCK_0
- U18 pad 38: /Teensy/TNY_CS_22 -> /Level Shifters/PAN3V.CS_22
- U18 pad 39: /Teensy/TNY_CS_21 -> /Level Shifters/PAN3V.CS_21
- U18 pad 4: /Teensy/TNY_CS_01 -> /Level Shifters/PAN3V.CS_01
- U18 pad 42: /Teensy/TNY_CS_20 -> /Level Shifters/PAN3V.CS_20
- U18 pad 43: /Teensy/TNY_CS_19 -> /Level Shifters/PAN3V.CS_19
- U18 pad 44: /Teensy/TNY_CS_18 -> /Level Shifters/PAN3V.CS_18
- U18 pad 45: /Teensy/TNY_CS_17 -> /Level Shifters/PAN3V.CS_17
- U18 pad 5: /Teensy/TNY_CS_02 -> /Level Shifters/PAN3V.CS_02
- U18 pad 6: /Teensy/TNY_CS_03 -> /Level Shifters/PAN3V.CS_03
- U18 pad 7: /Teensy/TNY_CS_04 -> /Level Shifters/PAN3V.CS_04
- U18 pad 8: /Teensy/TNY_CS_05 -> /Level Shifters/PAN3V.CS_05
- U18 pad 9: /Teensy/TNY_CS_06 -> /Level Shifters/PAN3V.CS_06
- U2 pad 1: /Level Shifters/PAN3V.MISO_0 -> /Level Shifters/PAN3V.CS_00
- U2 pad 2: GND -> +3.3V
- U2 pad 3: /Level Shifters/PAN3V.MISO_1 -> /Level Shifters/PAN3V.CS_01
- U2 pad 4: /Teensy/TNY_MISO_1 -> /Level Shifters/PAN3V.CS_02
- U2 pad 5: +3.3V -> /Level Shifters/PAN3V.CS_03
- U2 pad 6: /Teensy/TNY_MISO_0 -> /Level Shifters/PAN3V.CS_04
- U3 pad 1: Net-(U3-A1) -> /Level Shifters/PAN3V.CS_08
- U3 pad 12: Net-(U3-B8) -> /Level Shifters/PAN5V.CS_15
- U3 pad 13: Net-(U3-B7) -> /Level Shifters/PAN5V.CS_14
- U3 pad 14: Net-(U3-B6) -> /Level Shifters/PAN5V.CS_13
- U3 pad 15: unconnected-(U3-B5-Pad15) -> /Level Shifters/PAN5V.CS_12
- U3 pad 16: Net-(U3-B4) -> /Level Shifters/PAN5V.CS_11
- U3 pad 17: unconnected-(U3-B3-Pad17) -> /Level Shifters/PAN5V.CS_10
- U3 pad 18: Net-(U3-B2) -> /Level Shifters/PAN5V.CS_09
- U3 pad 20: Net-(U3-B1) -> /Level Shifters/PAN5V.CS_08
- U3 pad 3: Net-(U3-A1) -> /Level Shifters/PAN3V.CS_09
- U3 pad 4: unconnected-(U3-A3-Pad4) -> /Level Shifters/PAN3V.CS_10
- U3 pad 5: Net-(U3-A1) -> /Level Shifters/PAN3V.CS_11
- U3 pad 6: unconnected-(U3-A5-Pad6) -> /Level Shifters/PAN3V.CS_12
- U3 pad 7: Net-(U3-A1) -> /Level Shifters/PAN3V.CS_13
- U3 pad 8: Net-(U3-A1) -> /Level Shifters/PAN3V.CS_14
- U3 pad 9: Net-(U3-A1) -> /Level Shifters/PAN3V.CS_15
- U4 pad 1: Net-(U4-A1) -> /Level Shifters/PAN3V.CS_16
- U4 pad 12: Net-(U4-B8) -> /Level Shifters/PAN5V.CS_23
- U4 pad 13: Net-(U4-B7) -> /Level Shifters/PAN5V.CS_22
- U4 pad 14: Net-(U4-B6) -> /Level Shifters/PAN5V.CS_21
- U4 pad 15: unconnected-(U4-B5-Pad15) -> /Level Shifters/PAN5V.CS_20
- U4 pad 16: Net-(U4-B4) -> /Level Shifters/PAN5V.CS_19
- U4 pad 17: unconnected-(U4-B3-Pad17) -> /Level Shifters/PAN5V.CS_18
- U4 pad 18: Net-(U4-B2) -> /Level Shifters/PAN5V.CS_17
- U4 pad 20: Net-(U4-B1) -> /Level Shifters/PAN5V.CS_16
- U4 pad 3: Net-(U4-A1) -> /Level Shifters/PAN3V.CS_17
- U4 pad 4: unconnected-(U4-A3-Pad4) -> /Level Shifters/PAN3V.CS_18
- U4 pad 5: Net-(U4-A1) -> /Level Shifters/PAN3V.CS_19
- U4 pad 6: unconnected-(U4-A5-Pad6) -> /Level Shifters/PAN3V.CS_20
- U4 pad 7: Net-(U4-A1) -> /Level Shifters/PAN3V.CS_21
- U4 pad 8: Net-(U4-A1) -> /Level Shifters/PAN3V.CS_22
- U4 pad 9: Net-(U4-A1) -> /Level Shifters/PAN3V.CS_23
- U5 pad 1: Net-(U5-A1) -> /Level Shifters/PAN3V.CS_24
- U5 pad 12: Net-(U5-B8) -> /Level Shifters/PAN5V.EXT_INT
- U5 pad 13: Net-(U5-B7) -> unconnected-(U5-B7-Pad13)
- U5 pad 14: Net-(U5-B6) -> /Level Shifters/PAN5V.CS_29
- U5 pad 15: unconnected-(U5-B5-Pad15) -> /Level Shifters/PAN5V.CS_28
- U5 pad 16: Net-(U5-B4) -> /Level Shifters/PAN5V.CS_27
- U5 pad 17: unconnected-(U5-B3-Pad17) -> /Level Shifters/PAN5V.CS_26
- U5 pad 18: Net-(U5-B2) -> /Level Shifters/PAN5V.CS_25
- U5 pad 20: Net-(U5-B1) -> /Level Shifters/PAN5V.CS_24
- U5 pad 3: Net-(U5-A1) -> /Level Shifters/PAN3V.CS_25
- U5 pad 4: unconnected-(U5-A3-Pad4) -> /Level Shifters/PAN3V.CS_26
- U5 pad 5: Net-(U5-A1) -> /Level Shifters/PAN3V.CS_27
- U5 pad 6: unconnected-(U5-A5-Pad6) -> /Level Shifters/PAN3V.CS_28
- U5 pad 7: Net-(U5-A1) -> /Level Shifters/PAN3V.CS_29
- U5 pad 8: Net-(U5-A1) -> unconnected-(U5-A7-Pad8)
- U5 pad 9: Net-(U5-A1) -> /Level Shifters/PAN3V.EXT_INT
Routing:
- removed copper zone on In2.Cu, net +5V
- removed copper zone on In1.Cu, net GND
Other:
- outline, holes or cut-outs redrawn
- copper layers 6 -> 4
