File: development/arena_12-12/teensy4p1/teensy_arena_12-12_v0p2/power.kicad_sch (KiCad schematic)
At the start: 3 parts, among them J1 Barrel_Jack, J4 Barrel_Jack, SW1 SW_SPDT

Commit message: first step cleanup
Parts:
- J1, J4: DigiKey PN (none) -> CP-063AH-ND; LCSC PN (none) -> C2928097; MPN (none) -> PJ-063AH
- SW1: DigiKey PN (none) -> CKC5102-ND; LCSC PN (none) -> C2798743; MPN (none) -> L102021ML04Q
Other:
- company: (none) -> IORodeo for Reiserlab @ Janelia
- title: (none) -> 12-12 Teensy G4.1 Arena Modular LED Display
Changed lines of the file:
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@@
 	(generator_version "8.0")
 	(paper "USLetter")
+	(title_block
+		(title "12-12 Teensy G4.1 Arena Modular LED Display")
+		(date "2024-12-23")
+		(rev "v0.3")
+		(company "IORodeo for Reiserlab @ Janelia")
+	)
 	(junction
 		(at 90.17 48.26)
@@
 	(text "Power"
 		(exclude_from_sim no)
-		(at 115.189 21.082 0)
+		(at 133.35 23.876 0)
 		(effects
 			(font
-				(size 2.54 2.54)
+				(size 5.08 5.08)
 				(thickness 0.508)
 				(bold yes)
@@
 			)
 		)
-		(property "Datasheet" "~"
+		(property "Datasheet" "https://datasheet.octopart.com/PJ-063AH-Same-Sky-datasheet-181917378.pdf"
 			(at 102.87 46.736 0)
 			(effects
@@
 		)
 		(property "Description" ""
+			(at 104.14 45.72 0)
+			(effects
+				(font
+					(size 1.27 1.27)
+				)
+				(hide yes)
+			)
+		)
+		(property "DigiKey PN" "CP-063AH-ND"
+			(at 104.14 45.72 0)
+			(effects
+				(font
+					(size 1.27 1.27)
+				)
+				(hide yes)
+			)
+		)
+		(property "LCSC PN" "C2928097"
+			(at 104.14 45.72 0)
+			(effects
+				(font
+					(size 1.27 1.27)
+				)
+				(hide yes)
+			)
+		)
+		(property "MPN" "PJ-063AH"
 			(at 104.14 45.72 0)
 			(effects
@@
 			)
 		)
-		(property "Datasheet" "~"
+		(property "Datasheet" "https://datasheet.octopart.com/L102021ML04Q-C%26K-Components-datasheet-62111167.pdf"
 			(at 71.12 45.72 0)
 			(effects
@@
 		)
 		(property "Description" ""
+			(at 71.12 45.72 0)
+			(effects
+				(font
+					(size 1.27 1.27)
+				)
+				(hide yes)
+			)
+		)
+		(property "DigiKey PN" "CKC5102-ND"
+			(at 71.12 45.72 0)
+			(effects
+				(font
+					(size 1.27 1.27)
+				)
+				(hide yes)
+			)
+		)
+		(property "LCSC PN" "C2798743"
+			(at 71.12 45.72 0)
+			(effects
+				(font
+					(size 1.27 1.27)
+				)
+				(hide yes)
+			)
+		)
+		(property "MPN" "L102021ML04Q"
 			(at 71.12 45.72 0)
 			(effects
@@
 			)
 		)
-		(property "Datasheet" "~"
+		(property "Datasheet" "https://datasheet.octopart.com/PJ-063AH-Same-Sky-datasheet-181917378.pdf"
 			(at 102.87 83.566 0)
 			(effects
@@
 			(at 104.14 82.55 0)
 			(effects
+				(font
+					(size 1.27 1.27)
+				)
+				(hide yes)
+			)
+		)
+		(property "DigiKey PN" "CP-063AH-ND"
+			(at 104.14 82.55 0)
+			(effects
+				(font
+					(size 1.27 1.27)
+				)
+				(hide yes)
+			)
+		)
+		(property "LCSC PN" "C2928097"
+			(at 104.14 82.55 0)
+			(effects
+				(font
+					(size 1.27 1.27)
+				)
+				(hide yes)
+			)
+		)
+		(property "MPN" "PJ-063AH"
+			(at 104.14 82.55 0)
+			(effects
