File: development/arena_12-12/teensy4p1/teensy_arena_12-12_v0p2/teensy.kicad_sch (KiCad schematic)
At the start: 41 parts, among them J2 Conn_01x04, J3 Conn_01x04, U1 Teensy4.1, U2 74LVC2G17

Commit message: first step cleanup
Parts:
- C1: DigiKey PN (none) -> 1276-1001-2-ND; LCSC PN (none) -> C1525; MPN (none) -> CL05B104KO5NNNC
- J2, J3: DigiKey PN (none) -> 455-SM04B-SRSS-TBTR-ND; LCSC PN (none) -> C145956; MPN (none) -> SM04B-SRSS-TB
- R10, R11, R12, R13, R14, R15, R16, R17, R18, R19, R20, R21, R22, R23, R24, R25, R26, R27, R28, R29, R3, R30, R31, R32, R33, R34, R35, R36, R37, R38, R4, R5, R6, R7, R8, R9: LCSC PN (none) -> C25105; MPN (none) -> 0402WGF330JTCE
- U1: now not fitted
- U2: DigiKey PN (none) -> 296-SN74LVC2G17DBVRTR-ND; LCSC PN (none) -> C10429; MPN (none) -> SN74LVC2G17DBVR
Other:
- company: (none) -> IORodeo for Reiserlab @ Janelia
- title: (none) -> 12-12 Teensy G4.1 Arena Modular LED Display
