File: development/arena_12-12/teensy4p1/teensy_arena_12-12_v0p2/teensy_arena_12-12.kicad_sch (KiCad schematic)
At the start: 0 parts

Commit message: first step cleanup
Other:
- company: (none) -> IORodeo for Reiserlab @ Janelia
- title: (none) -> 12-12 Teensy G4.1 Arena Modular LED Display
Changed lines of the file:
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@@
 	(generator "eeschema")
 	(generator_version "8.0")
-	(paper "User" 279.4 203.2)
+	(paper "USLetter")
 	(title_block
-		(date "11 jun 2015")
+		(title "12-12 Teensy G4.1 Arena Modular LED Display")
+		(date "2024-12-23")
+		(rev "v0.3")
+		(company "IORodeo for Reiserlab @ Janelia")
 	)
 	(bus
