File: development/arena_12-12/teensy4p1/teensy_arena_12-12_v0p3/level_shifters.kicad_sch (KiCad schematic)
At the start: 166 parts, among them U10 TXB0108PW, U11 TXB0108PW, U12 TXB0108PW, U13 TXB0108PW, U14 TXB0108PW, U15 74LVC1G17, U16 74LVC1G17, U17 74LVC1G17, U18 74LVC1G17, U19 74LVC2G17, U20 74LVC2G17, U21 74LVC2G17, U22 74LVC2G17, U23 74LVC2G17, U24 74LVC2G17, U25 74LVC2G17, U26 74LVC2G17, U27 74LVC2G17, U28 74LVC2G17, U29 74LVC2G17, U3 TXB0108PW, U30 74LVC2G17, U31 74LVC2G17, U32 74LVC2G17, U33 74LVC2G17, U34 74LVC2G17, U35 74LVC2G17, U4 TXB0108PW, U5 TXB0108PW, U6 TXB0108PW, U7 TXB0108PW, U8 TXB0108PW, U9 TXB0108PW

Commit message: export for production
Parts:
- C10, C11, C12, C13, C14, C15, C16, C17, C18, C19, C2, C20, C21, C22, C23, C24, C25, C26, C27, C28, C29, C3, C30, C31, C32, C33, C34, C35, C36, C37, C38, C39, C4, C40, C41, C42, C43, C44, C45, C46, C5, C6, C7, C8, C9: LCSC PN C1525 -> (none); LCSC Part # (none) -> C1525
- R100, R101, R102, R103, R104, R105, R106, R107, R108, R109, R110, R111, R112, R113, R114, R115, R116, R117, R118, R119, R120, R121, R122, R123, R124, R125, R126, R39, R40, R41, R42, R43, R44, R45, R46, R47, R48, R49, R50, R51, R52, R53, R54, R55, R56, R57, R58, R59, R60, R61, R62, R63, R64, R65, R66, R67, R68, R69, R70, R71, R72, R73, R74, R75, R76, R77, R78, R79, R80, R81, R82, R83, R84, R85, R86, R87, R88, R89, R90, R91, R92, R93, R94, R95, R96, R97, R98, R99: LCSC PN C25105 -> (none); LCSC Part # (none) -> C25105
- U10, U11, U12, U13, U14, U3, U4, U5, U6, U7, U8, U9: LCSC PN C53406 -> (none); LCSC Part # (none) -> C53406
- U15, U16, U17, U18: LCSC PN C7836 -> (none); LCSC Part # (none) -> C7836
- U19, U20, U21, U22, U23, U24, U25, U26, U27, U28, U29, U30, U31, U32, U33, U34, U35: LCSC PN C10429 -> (none); LCSC Part # (none) -> C10429
