File: development/arena_12-12/teensy4p1/teensy_arena_12-12_v0p3/panel_headers.kicad_sch (KiCad schematic)
At the start: 231 parts, among them P1 CONN15, P10 CONN15, P11 CONN15, P12 CONN15, P2 CONN15, P3 CONN15, P4 CONN15, P5 CONN15, P6 CONN15, P7 CONN15, P8 CONN15, P9 CONN15, Q1 MOSFET_NCHAN, U36 74LVC2G17, U37 74LVC2G17, U38 74LVC2G17, U39 74LVC2G17, U40 74LVC2G17, U41 74LVC2G17, U42 74LVC2G17, U43 74LVC2G17, U44 74LVC2G17, U45 74LVC2G17, U46 74LVC2G17, U47 74LVC2G17, U48 74LVC2G17, U49 74LVC2G17, U50 74LVC2G17, U51 74LVC2G17, U52 74LVC2G17, U53 74LVC2G17, U54 74LVC2G17, U55 74LVC2G17, U56 74LVC2G17, U57 74LVC2G17, U58 74LVC2G17, U59 74LVC2G17, U60 74LVC2G17, U61 74LVC2G17, U62 74LVC2G17, U63 74LVC2G17, U64 74LVC2G17, U65 74LVC2G17, U66 74LVC2G17, U67 74LVC2G17, U68 74LVC2G17, U69 74LVC2G17, U70 74LVC2G17, U71 74LVC2G17, U72 74LVC2G17, U73 74LVC2G17, U74 74LVC2G17, U75 74LVC2G17, U76 74LVC2G17, U77 74LVC2G17, U78 74LVC2G17, U79 74LVC2G17, U80 74LVC2G17, U81 74LVC2G17, U82 74LVC2G17, U83 74LVC2G17

Commit message: export for production
Parts:
- C100, C101, C102, C103, C104, C105, C106, C95, C96, C97, C98, C99: LCSC PN C7432790 -> (none); LCSC Part # (none) -> C7432790
- C47, C48, C49, C50, C51, C52, C53, C54, C55, C56, C57, C58, C59, C60, C61, C62, C63, C64, C65, C66, C67, C68, C69, C70, C71, C72, C73, C74, C75, C76, C77, C78, C79, C80, C81, C82, C83, C84, C85, C86, C87, C88, C89, C90, C91, C92, C93, C94: LCSC PN C1525 -> (none); LCSC Part # (none) -> C1525
- P1, P10, P11, P12, P2, P3, P4, P5, P6, P7, P8, P9: LCSC PN C5210739 -> (none); LCSC Part # (none) -> C18078136
- Q1: LCSC PN C165220 -> (none); LCSC Part # (none) -> C165220
- R1: LCSC PN C25087 -> (none); LCSC Part # (none) -> C25087
- R127, R128, R129, R130, R131, R132, R133, R134, R135, R136, R137, R138, R139, R140, R141, R142, R143, R144, R145, R146, R147, R148, R149, R150, R151, R152, R153, R154, R155, R156, R157, R158, R159, R160, R161, R162, R163, R164, R165, R166, R167, R168, R169, R170, R171, R172, R173, R174, R175, R176, R177, R178, R179, R180, R181, R182, R183, R184, R185, R186, R187, R188, R189, R190, R191, R192, R193, R194, R195, R196, R197, R198, R199, R200, R201, R202, R203, R204, R205, R206, R207, R208, R209, R210, R211, R212, R213, R214, R215, R216, R217, R218, R219, R220, R221, R222, R223, R224, R225, R226, R227, R228, R229, R230, R231, R232, R233, R234: LCSC PN C25105 -> (none); LCSC Part # (none) -> C25105
- R2: LCSC PN C25765 -> (none); LCSC Part # (none) -> C25765
- U36, U37, U38, U39, U40, U41, U42, U43, U44, U45, U46, U47, U48, U49, U50, U51, U52, U53, U54, U55, U56, U57, U58, U59, U60, U61, U62, U63, U64, U65, U66, U67, U68, U69, U70, U71, U72, U73, U74, U75, U76, U77, U78, U79, U80, U81, U82, U83: LCSC PN C10429 -> (none); LCSC Part # (none) -> C10429
