File: development/arena_12-12/teensy4p1/teensy_arena_12-12_v0p3/power.kicad_sch (KiCad schematic)
At the start: 3 parts, among them J1 Barrel_Jack, J4 Barrel_Jack, SW1 SW_SPDT

Commit message: export for production
Parts:
- J1, J4: LCSC PN C2928097 -> (none); LCSC Part # (none) -> C2928097
- SW1: LCSC PN C2798743 -> (none); LCSC Part # (none) -> C2798743
Changed lines of the file:
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@@
 			)
 		)
-		(property "LCSC PN" "C2928097"
+		(property "MPN" "PJ-063AH"
 			(at 104.14 45.72 0)
 			(effects
@@
 			)
 		)
-		(property "MPN" "PJ-063AH"
+		(property "LCSC Part #" "C2928097"
 			(at 104.14 45.72 0)
 			(effects
@@
 			)
 		)
-		(property "LCSC PN" "C2798743"
+		(property "MPN" "L102021ML04Q"
 			(at 71.12 45.72 0)
 			(effects
@@
 			)
 		)
-		(property "MPN" "L102021ML04Q"
+		(property "LCSC Part #" "C2798743"
 			(at 71.12 45.72 0)
 			(effects
@@
 			)
 		)
-		(property "LCSC PN" "C2928097"
-			(at 104.14 82.55 0)
-			(effects
-				(font
-					(size 1.27 1.27)
-				)
-				(hide yes)
-			)
-		)
 		(property "MPN" "PJ-063AH"
 			(at 104.14 82.55 0)
 			(effects
+				(font
+					(size 1.27 1.27)
+				)
+				(hide yes)
+			)
+		)
+		(property "LCSC Part #" "C2928097"
+			(at 104.14 82.55 0)
+			(effects
