File: development/arena_12-12/teensy4p1/teensy_arena_12-12_v0p3/teensy.kicad_sch (KiCad schematic)
At the start: 41 parts, among them J2 Conn_01x04, J3 Conn_01x04, U1 Teensy4.1, U2 74LVC2G17

Commit message: export for production
Parts:
- C1: LCSC PN C1525 -> (none); LCSC Part # (none) -> C1525
- J2, J3: LCSC PN C145956 -> (none); LCSC Part # (none) -> C145956
- R10, R11, R12, R13, R14, R15, R16, R17, R18, R19, R20, R21, R22, R23, R24, R25, R26, R27, R28, R29, R3, R30, R31, R32, R33, R34, R35, R36, R37, R38, R4, R5, R6, R7, R8, R9: LCSC PN C25105 -> (none); LCSC Part # (none) -> C25105
- U2: LCSC PN C10429 -> (none); LCSC Part # (none) -> C10429
