File: development/arena_12-12/top/arena_top_12-12/arena_top_12-12.kicad_pcb (KiCad board)
At the start: 2 copper layers, 228.6 x 228.6 mm, 41 parts, among them J4 Barrel_Jack, P1 CONN15, P10 CONN15, P11 CONN15, P12 CONN15, P2 CONN15, P3 CONN15, P4 CONN15, P5 CONN15, P6 CONN15, P7 CONN15, P8 CONN15, P9 CONN15

Commit message: export for production
Other:
- board text added: "12-12 Teensy G4.1 Arena Top v0.3.3"
- board text added: "2024-12-23"
- board text added: "https://reiserlab.github.io/Modular-LED-Display/"
- board text removed: "Teensy 12-12 Arena-Top V0.1 R1"
