File: development/arena_12-12/top/arena_top_12-12/panel_headers.kicad_sch (KiCad schematic)
At the start: 36 parts, among them P1 CONN15, P10 CONN15, P11 CONN15, P12 CONN15, P2 CONN15, P3 CONN15, P4 CONN15, P5 CONN15, P6 CONN15, P7 CONN15, P8 CONN15, P9 CONN15

Commit message: export for production
Parts:
- C1, C10, C11, C12, C2, C3, C4, C5, C6, C7, C8, C9: LCSC Part # (none) -> C7432790; MPN (none) -> HGC1210R5107M160NSVK
- C13, C14, C15, C16, C17, C18, C19, C20, C21, C22, C23, C24: DigiKey PN (none) -> 1189-1856-ND; LCSC Part # (none) -> C338173; MPN (none) -> 16YXF100MEFC6.3X11
- P1, P10, P11, P12, P2, P3, P4, P5, P6, P7, P8, P9: DigiKey PN (none) -> S1011EC-40-ND; LCSC Part # (none) -> C7501269; MPN (none) -> PRPC040SAAN-RC
