File: development/arena_12-12/top/arena_top_12-12/power.kicad_sch (KiCad schematic)
At the start: 1 part, among them J4 Barrel_Jack

Commit message: export for production
Parts:
- J4: DigiKey PN (none) -> CP-063AH-ND; LCSC Part # (none) -> C2928097; MPN (none) -> PJ-063AH
Changed lines of the file:
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@@
 			)
 		)
-		(property "Datasheet" "~"
+		(property "Datasheet" "https://octopart.com/datasheet/pj-063ah-same+sky-106234056"
 			(at 102.87 83.566 0)
 			(effects
@@
 			(at 104.14 82.55 0)
 			(effects
+				(font
+					(size 1.27 1.27)
+				)
+				(hide yes)
+			)
+		)
+		(property "DigiKey PN" "CP-063AH-ND"
+			(at 104.14 82.55 0)
+			(effects
+				(font
+					(size 1.27 1.27)
+				)
+				(hide yes)
+			)
+		)
+		(property "LCSC Part #" "C2928097"
+			(at 104.14 82.55 0)
+			(effects
+				(font
+					(size 1.27 1.27)
+				)
+				(hide yes)
+			)
+		)
+		(property "MPN" "PJ-063AH"
+			(at 104.14 82.55 0)
+			(effects
